File: Wooden_Mirror.kicad_pcb (KiCad board)
At the start: 2 copper layers, 18 x 80.8 mm, 2 parts, among them J1 Conn_02x10_Odd_Even, J5 Conn_02x10_Odd_Even

Commit message: 2nd try
Parts:
- moved J1 12.7 mm to (91.4, 124.5)
Routing:
- net /LED_DIN: track 78.8 -> 91.5 mm
- net Net-(J1-Pin_19): track 82.5 -> 95.1 mm
- net /Serial_IN: track 77.4 -> 88.9 mm
- net Net-(J1-Pin_17): track 74.5 -> 85.9 mm
Other:
- board size 18 x 80.8 mm -> 18 x 93.5 mm
Changed lines of the file:
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@@
 	(footprint "Connector_PinHeader_2.54mm:PinHeader_2x10_P2.54mm_Vertical"
 		(layer "F.Cu")
-		(at 91.44 111.76)
+		(at 91.44 124.46)
 		(descr "Through hole straight pin header, 2x10, 2.54mm pitch, double rows")
 		(tags "Through hole pin header THT 2x10 2.54mm double row")
@@
 	)
 	(gr_line
-		(start 88.9 121.92)
-		(end 88.9 129.54)
+		(start 88.265 134.62)
+		(end 88.265 142.24)
 		(stroke
 			(width 0.15)
@@
 	)
 	(gr_line
-		(start 88.9 119.38)
-		(end 89.535 119.38)
+		(start 88.265 132.08)
+		(end 88.9 132.08)
 		(stroke
 			(width 0.15)
@@
 	)
 	(gr_line
-		(start 88.9 129.54)
-		(end 89.535 129.54)
+		(start 88.265 142.24)
+		(end 88.9 142.24)
 		(stroke
 			(width 0.15)
@@
 	)
 	(gr_line
-		(start 89.535 111.76)
-		(end 88.9 111.76)
-		(stroke
-			(width 0.15)
-			(type default)
-		)
-		(layer "F.SilkS")
-	)
-	(gr_line
-		(start 89.535 121.92)
-		(end 88.9 121.92)
+		(start 88.9 124.46)
+		(end 88.265 124.46)
+		(stroke
+			(width 0.15)
+			(type default)
+		)
+		(layer "F.SilkS")
+	)
+	(gr_line
+		(start 88.9 134.62)
+		(end 88.265 134.62)
 		(stroke
 			(width 0.15)
@@
 	)
 	(gr_line
-		(start 88.9 111.76)
-		(end 88.9 119.38)
+		(start 88.265 124.46)
+		(end 88.265 132.08)
 		(stroke
 			(width 0.15)
@@
 	)
 	(gr_rect
-		(start 83.82 57.404)
-		(end 101.854 138.176)
+		(start 83.82 57.277)
+		(end 101.854 150.749)
 		(stroke
 			(width 0.1)
@@
 	)
 	(gr_text "GND"
-		(at 85.09 116.205 0)
+		(at 84.455 128.905 0)
 		(layer "F.SilkS")
 		(effects
@@
 	)
 	(gr_text "+5V"
-		(at 85.09 126.365 0)
+		(at 84.455 139.065 0)
 		(layer "F.SilkS")
 		(effects
@@
 	)
 	(segment
+		(start 97.155 144.145)
+		(end 93.98 147.32)
+		(width 0.25)
+		(layer "F.Cu")
+		(net 3)
+	)
+	(segment
+		(start 91.44 60.96)
+		(end 92.615 62.135)
+		(width 0.25)
+		(layer "F.Cu")
+		(net 3)
+	)
+	(segment
+		(start 92.615 62.135)
+		(end 95.155 62.135)
+		(width 0.25)
+		(layer "F.Cu")
+		(net 3)
+	)
+	(segment
 		(start 97.155 64.135)
-		(end 95.155 62.135)
+		(end 97.155 144.145)
 		(width 0.25)
 		(layer "F.Cu")
@@
 	)
 	(segment
-		(start 92.615 62.135)
-		(end 91.44 60.96)
+		(start 95.155 62.135)
+		(end 97.155 64.135)
 		(width 0.25)
 		(layer "F.Cu")
 		(net 3)
-	)
-	(segment
-		(start 95.155 62.135)
-		(end 92.615 62.135)
-		(width 0.25)
-		(layer "F.Cu")
-		(net 3)
-	)
-	(segment
-		(start 97.155 131.445)
-		(end 97.155 64.135)
-		(width 0.25)
-		(layer "F.Cu")
-		(net 3)
-	)
-	(segment
-		(start 93.98 134.62)
-		(end 97.155 131.445)
-		(width 0.25)
-		(layer "F.Cu")
-		(net 3)
-	)
-	(segment
-		(start 97.155 66.675)
-		(end 97.155 130.175)
-		(width 0.25)
-		(layer "B.Cu")
-		(net 4)
 	)
 	(segment
@@
 	)
 	(segment
-		(start 92.615 130.905)
-		(end 91.44 132.08)
+		(start 97.155 140.726701)
+		(end 94.371701 143.51)
 		(width 0.25)
 		(layer "B.Cu")
@@
 	)
 	(segment
-		(start 97.155 130.175)
-		(end 96.425 130.905)
+		(start 97.155 66.675)
+		(end 97.155 140.726701)
 		(width 0.25)
 		(layer "B.Cu")
@@
 	)
 	(segment
-		(start 96.425 130.905)
-		(end 92.615 130.905)
+		(start 94.371701 143.51)
+		(end 92.71 143.51)
 		(width 0.25)
 		(layer "B.Cu")
@@
 	)
 	(segment
-		(start 92.71 135.89)
-		(end 91.44 134.62)
+		(start 92.71 143.51)
+		(end 91.44 144.78)
+		(width 0.25)
+		(layer "B.Cu")
+		(net 4)
+	)
+	(segment
+		(start 92.615 148.495)
+		(end 91.44 147.32)
 		(width 0.25)
 		(layer "F.Cu")
@@
 	)
 	(segment
-		(start 97.79 132.471701)
-		(end 94.371701 135.89)
+		(start 93.98 60.96)
+		(end 95.885 60.96)
+		(width 0.25)
+		(layer "F.Cu")
+		(net 5)
+	)
+	(segment
+		(start 94.466701 148.495)
+		(end 92.615 148.495)
 		(width 0.25)
 		(layer "F.Cu")
@@
 	)
 	(segment
-		(start 94.371701 135.89)
-		(end 92.71 135.89)
+		(start 97.79 62.865)
+		(end 97.79 145.171701)
 		(width 0.25)
 		(layer "F.Cu")
@@
 	)
 	(segment
-		(start 93.98 60.96)
-		(end 95.885 60.96)
+		(start 97.79 145.171701)
+		(end 94.466701 148.495)
 		(width 0.25)
 		(layer "F.Cu")
@@
 	)
 	(segment
-		(start 97.79 62.865)
-		(end 97.79 132.471701)
-		(width 0.25)
-		(layer "F.Cu")
-		(net 5)
-	)
-	(segment
-		(start 97.79 130.176396)
+		(start 97.79 140.97)
+		(end 93.98 144.78)
+		(width 0.25)
+		(layer "B.Cu")
+		(net 6)
+	)
+	(segment
+		(start 92.6338 62.3062)
+		(end 94.447901 62.3062)
+		(width 0.25)
+		(layer "B.Cu")
+		(net 6)
+	)
+	(segment
+		(start 91.44 63.5)
+		(end 92.6338 62.3062)
+		(width 0.25)
+		(layer "B.Cu")
+		(net 6)
+	)
+	(segment
+		(start 97.79 65.648299)
+		(end 97.79 140.97)
+		(width 0.25)
+		(layer "B.Cu")
+		(net 6)
+	)
+	(segment
+		(start 94.447901 62.3062)
 		(end 97.79 65.648299)
-		(width 0.25)
-		(layer "B.Cu")
-		(net 6)
-	)
-	(segment
-		(start 94.447901 62.3062)
-		(end 92.6338 62.3062)
-		(width 0.25)
-		(layer "B.Cu")
-		(net 6)
-	)
-	(segment
-		(start 92.6338 62.3062)
-		(end 91.44 63.5)
-		(width 0.25)
-		(layer "B.Cu")
-		(net 6)
-	)
-	(segment
-		(start 95.886396 132.08)
-		(end 97.79 130.176396)
-		(width 0.25)
-		(layer "B.Cu")
-		(net 6)
-	)
-	(segment
-		(start 93.98 132.08)
-		(end 95.886396 132.08)
-		(width 0.25)
-		(layer "B.Cu")
-		(net 6)
-	)
-	(segment
-		(start 97.79 65.648299)
-		(end 94.447901 62.3062)
 		(width 0.25)
 		(layer "B.Cu")
@@
 		(polygon
 			(pts
-				(xy 84.328 57.911697) (xy 84.328 137.667697) (xy 101.346 137.667697) (xy 101.346 57.912)
+				(xy 84.328 57.911697) (xy 84.328 150.367697) (xy 101.346 150.367697) (xy 101.346 57.912)
 			)
 		)
@@
 		(polygon
 			(pts
-				(xy 84.328 57.912) (xy 84.328 137.668) (xy 101.346 137.668) (xy 101.346 57.912)
-			)
-		)
+				(xy 84.328 57.912) (xy 84.328 150.368) (xy 101.346 150.368) (xy 101.346 57.912)
+			)
+		)

Commit message: updated
Parts:
- moved J1 15.2 mm to (91.4, 109.2)
- moved J5 15.2 mm to (94.0, 68.6)
Other:
- board size 18 x 93.5 mm -> 18 x 119.4 mm
Changed lines of the file:
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@@
 	(footprint "Connector_PinHeader_2.54mm:PinHeader_2x10_P2.54mm_Vertical"
 		(layer "F.Cu")
-		(at 93.98 83.82 180)
+		(at 93.98 68.58 180)
 		(descr "Through hole straight pin header, 2x10, 2.54mm pitch, double rows")
 		(tags "Through hole pin header THT 2x10 2.54mm double row")
@@
 	(footprint "Connector_PinHeader_2.54mm:PinHeader_2x10_P2.54mm_Vertical"
 		(layer "F.Cu")
-		(at 91.44 124.46)
+		(at 91.44 109.22)
 		(descr "Through hole straight pin header, 2x10, 2.54mm pitch, double rows")
 		(tags "Through hole pin header THT 2x10 2.54mm double row")
@@
 	)
 	(gr_line
-		(start 88.265 134.62)
-		(end 88.265 142.24)
+		(start 88.265 119.38)
+		(end 88.265 127)
 		(stroke
 			(width 0.15)
@@
 	)
 	(gr_line
-		(start 88.9 73.66)
-		(end 89.535 73.66)
+		(start 88.9 58.42)
+		(end 89.535 58.42)
 		(stroke
 			(width 0.15)
@@
 	)
 	(gr_line
-		(start 88.265 132.08)
-		(end 88.9 132.08)
+		(start 88.265 116.84)
+		(end 88.9 116.84)
 		(stroke
 			(width 0.15)
@@
 	)
 	(gr_line
-		(start 88.9 76.2)
-		(end 88.9 83.82)
+		(start 88.9 60.96)
+		(end 88.9 68.58)
 		(stroke
 			(width 0.15)
@@
 	)
 	(gr_line
-		(start 88.9 66.04)
-		(end 88.9 73.66)
+		(start 88.9 50.8)
+		(end 88.9 58.42)
 		(stroke
 			(width 0.15)
@@
 	)
 	(gr_line
-		(start 88.265 142.24)
-		(end 88.9 142.24)
+		(start 88.265 127)
+		(end 88.9 127)
 		(stroke
 			(width 0.15)
@@
 	)
 	(gr_line
-		(start 89.535 76.2)
-		(end 88.9 76.2)
+		(start 89.535 60.96)
+		(end 88.9 60.96)
 		(stroke
 			(width 0.15)
@@
 	)
 	(gr_line
-		(start 88.9 124.46)
-		(end 88.265 124.46)
+		(start 88.9 109.22)
+		(end 88.265 109.22)
 		(stroke
 			(width 0.15)
@@
 	)
 	(gr_line
-		(start 88.9 134.62)
-		(end 88.265 134.62)
+		(start 88.9 119.38)
+		(end 88.265 119.38)
 		(stroke
 			(width 0.15)
@@
 	)
 	(gr_line
-		(start 89.535 66.04)
-		(end 88.9 66.04)
+		(start 89.535 50.8)
+		(end 88.9 50.8)
 		(stroke
 			(width 0.15)
@@
 	)
 	(gr_line
-		(start 88.265 124.46)
-		(end 88.265 132.08)
+		(start 88.265 109.22)
+		(end 88.265 116.84)
 		(stroke
 			(width 0.15)
@@
 	)
 	(gr_line
-		(start 88.9 83.82)
-		(end 89.535 83.82)
+		(start 88.9 68.58)
+		(end 89.535 68.58)
 		(stroke
 			(width 0.15)
@@
 	)
 	(gr_rect
-		(start 83.82 57.277)
-		(end 101.854 150.749)
+		(start 83.82 29.21)
+		(end 101.854 148.59)
 		(stroke
 			(width 0.1)
@@
 	)
 	(gr_text "GND"
-		(at 84.455 128.905 0)
+		(at 84.455 126.365 0)
 		(layer "F.SilkS")
 		(effects
@@
 	)
 	(gr_text "\nInput"
-		(at 96.52 132.08 0)
+		(at 96.52 116.84 0)
 		(layer "F.SilkS")
 		(effects
@@
 	)
 	(gr_text "+5V"
-		(at 85.09 70.485 0)
+		(at 85.09 55.245 0)
 		(layer "F.SilkS")
 		(effects
@@
 	)
 	(gr_text "GND"
-		(at 85.0646 80.6196 0)
+		(at 85.0646 65.3796 0)
 		(layer "F.SilkS")
 		(effects
@@
 	)
 	(gr_text "+5V"
-		(at 84.455 139.065 0)
+		(at 84.328 113.538 0)
 		(layer "F.SilkS")
 		(effects
@@
 	)
 	(gr_text "EGS 1006 \nConnector"
-		(at 95.504 93.218 180)
+		(at 95.504 77.978 180)
 		(layer "F.SilkS")
 		(effects
@@
 	)
 	(gr_text "\nOutput"
-		(at 84.074 63.5 0)
+		(at 96.266 60.452 0)
 		(layer "F.SilkS")
 		(effects
@@
 	)
 	(gr_text "EGS 1006 \nConnector"
-		(at 87.884 100.33 0)
+		(at 87.884 85.09 0)
 		(layer "F.SilkS")
 		(effects
@@
 	)
 	(segment
-		(start 97.155 144.145)
-		(end 93.98 147.32)
+		(start 97.155 128.905)
+		(end 93.98 132.08)
 		(width 0.25)
 		(layer "F.Cu")
@@
 	)
 	(segment
-		(start 91.44 60.96)
-		(end 92.615 62.135)
+		(start 91.44 45.72)
+		(end 92.615 46.895)
 		(width 0.25)
 		(layer "F.Cu")
@@
 	)
 	(segment
-		(start 92.615 62.135)
-		(end 95.155 62.135)
+		(start 92.615 46.895)
+		(end 95.155 46.895)
 		(width 0.25)
 		(layer "F.Cu")
@@
 	)
 	(segment
-		(start 97.155 64.135)
-		(end 97.155 144.145)
+		(start 97.155 48.895)
+		(end 97.155 128.905)
 		(width 0.25)
 		(layer "F.Cu")
@@
 	)
 	(segment
-		(start 95.155 62.135)
-		(end 97.155 64.135)
+		(start 95.155 46.895)
+		(end 97.155 48.895)
 		(width 0.25)
 		(layer "F.Cu")
@@
 	)
 	(segment
-		(start 93.98 63.5)
-		(end 97.155 66.675)
+		(start 93.98 48.26)
+		(end 97.155 51.435)
 		(width 0.25)
 		(layer "B.Cu")
@@
 	)
 	(segment
-		(start 97.155 140.726701)
-		(end 94.371701 143.51)
+		(start 97.155 125.486701)
+		(end 94.371701 128.27)
 		(width 0.25)
 		(layer "B.Cu")
@@
 	)
 	(segment
-		(start 97.155 66.675)
-		(end 97.155 140.726701)
+		(start 97.155 51.435)
+		(end 97.155 125.486701)
 		(width 0.25)
 		(layer "B.Cu")
@@
 	)
 	(segment
-		(start 94.371701 143.51)
-		(end 92.71 143.51)
+		(start 94.371701 128.27)
+		(end 92.71 128.27)
 		(width 0.25)
 		(layer "B.Cu")
@@
 	)
 	(segment
-		(start 92.71 143.51)
-		(end 91.44 144.78)
+		(start 92.71 128.27)
+		(end 91.44 129.54)
 		(width 0.25)
 		(layer "B.Cu")
@@
 	)
 	(segment
-		(start 92.615 148.495)
-		(end 91.44 147.32)
+		(start 92.615 133.255)
+		(end 91.44 132.08)
 		(width 0.25)
 		(layer "F.Cu")
@@
 	)
 	(segment
-		(start 93.98 60.96)
-		(end 95.885 60.96)
+		(start 93.98 45.72)
+		(end 95.885 45.72)
 		(width 0.25)
 		(layer "F.Cu")
@@
 	)
 	(segment
-		(start 94.466701 148.495)
-		(end 92.615 148.495)
+		(start 94.466701 133.255)
+		(end 92.615 133.255)
 		(width 0.25)
 		(layer "F.Cu")
@@
 	)
 	(segment
-		(start 95.885 60.96)
-		(end 97.79 62.865)
+		(start 95.885 45.72)
+		(end 97.79 47.625)
 		(width 0.25)
 		(layer "F.Cu")
@@
 	)
 	(segment
-		(start 97.79 62.865)
-		(end 97.79 145.171701)
+		(start 97.79 47.625)
+		(end 97.79 129.931701)
 		(width 0.25)
 		(layer "F.Cu")
@@
 	)
 	(segment
-		(start 97.79 145.171701)
-		(end 94.466701 148.495)
+		(start 97.79 129.931701)
+		(end 94.466701 133.255)
 		(width 0.25)
 		(layer "F.Cu")
@@
 	)
 	(segment
-		(start 97.79 140.97)
-		(end 93.98 144.78)
+		(start 97.79 125.73)
+		(end 93.98 129.54)
 		(width 0.25)
 		(layer "B.Cu")
@@
 	)
 	(segment
-		(start 92.6338 62.3062)
-		(end 94.447901 62.3062)
+		(start 92.6338 47.0662)
+		(end 94.447901 47.0662)
 		(width 0.25)
 		(layer "B.Cu")
@@
 	)
 	(segment
-		(start 91.44 63.5)
-		(end 92.6338 62.3062)
+		(start 91.44 48.26)
+		(end 92.6338 47.0662)
 		(width 0.25)
 		(layer "B.Cu")
@@
 	)
 	(segment
-		(start 97.79 65.648299)
-		(end 97.79 140.97)
+		(start 97.79 50.408299)
+		(end 97.79 125.73)
 		(width 0.25)
 		(layer "B.Cu")
@@
 	)
 	(segment
-		(start 94.447901 62.3062)
-		(end 97.79 65.648299)
+		(start 94.447901 47.0662)
+		(end 97.79 50.408299)
 		(width 0.25)
 		(layer "B.Cu")
@@
 		(polygon
 			(pts
-				(xy 84.328 57.911697) (xy 84.328 150.367697) (xy 101.346 150.367697) (xy 101.346 57.912)
+				(xy 84.074 29.718) (xy 84.201 148.335697) (xy 101.6 148.335697) (xy 101.6 29.718)
 			)
 		)
@@
 		(polygon
 			(pts
-				(xy 84.328 57.912) (xy 84.328 150.368) (xy 101.346 150.368) (xy 101.346 57.912)
-			)
-		)
+				(xy 84.074 29.718) (xy 84.201 148.335932) (xy 101.6 148.336) (xy 101.6 29.718)
+			)
+		)
