File: Wooden_Mirror.kicad_pcb (KiCad board)
At the start: 2 copper layers, 18 x 119.4 mm, 2 parts, among them J1 Conn_02x10_Odd_Even, J5 Conn_02x10_Odd_Even

Commit message: nkmlkl
Parts:
- added H1: MH, MountingHole:MountingHole_3.2mm_M3_Pad, F.Cu at (91.4, 34.3)
- added H2: MH, MountingHole:MountingHole_3.2mm_M3_Pad, F.Cu at (91.4, 76.2)
- added H3: MH, MountingHole:MountingHole_3.2mm_M3_Pad, F.Cu at (91.4, 99.1)
- added H4: MH, MountingHole:MountingHole_3.2mm_M3_Pad, F.Cu at (91.4, 143.5)
- moved J5 1.80 mm to (92.7, 67.3)
- moved J1 1.80 mm to (90.2, 108.0)

Commit message: mnm,
Parts:
- moved H3 33.0 mm to (58.4, 99.1)
- moved H2 19.0 mm to (91.4, 95.2)
Changed lines of the file:
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@@
 	(footprint "MountingHole:MountingHole_3.2mm_M3_Pad"
 		(layer "F.Cu")
-		(at 91.44 99.06)
+		(at 58.42 99.06)
 		(descr "Mounting Hole 3.2mm, M3")
 		(tags "mounting hole 3.2mm m3")
@@
 	(footprint "MountingHole:MountingHole_3.2mm_M3_Pad"
 		(layer "F.Cu")
-		(at 91.44 76.2)
+		(at 91.44 95.25)
 		(descr "Mounting Hole 3.2mm, M3")
 		(tags "mounting hole 3.2mm m3")

Commit message: jiok
Parts:
- moved H3 38.8 mm to (91.4, 78.7)
- moved H2 1.27 mm to (91.4, 96.5)
- moved J1 1.27 mm to (90.2, 109.2)
- moved J5 1.27 mm to (92.7, 68.6)
Changed lines of the file:
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@@
 	(footprint "Connector_PinHeader_2.54mm:PinHeader_2x10_P2.54mm_Vertical"
 		(layer "F.Cu")
-		(at 92.71 67.31 180)
+		(at 92.71 68.58 180)
 		(descr "Through hole straight pin header, 2x10, 2.54mm pitch, double rows")
 		(tags "Through hole pin header THT 2x10 2.54mm double row")
@@
 	(footprint "Connector_PinHeader_2.54mm:PinHeader_2x10_P2.54mm_Vertical"
 		(layer "F.Cu")
-		(at 90.17 107.95)
+		(at 90.17 109.22)
 		(descr "Through hole straight pin header, 2x10, 2.54mm pitch, double rows")
 		(tags "Through hole pin header THT 2x10 2.54mm double row")
@@
 	(footprint "MountingHole:MountingHole_3.2mm_M3_Pad"
 		(layer "F.Cu")
-		(at 58.42 99.06)
+		(at 91.44 78.74)
 		(descr "Mounting Hole 3.2mm, M3")
 		(tags "mounting hole 3.2mm m3")
@@
 		)
 		(property "Value" "MH"
-			(at 0 4.2 0)
+			(at 0 5.47 0)
 			(layer "F.Fab")
 			(effects
@@
 	(footprint "MountingHole:MountingHole_3.2mm_M3_Pad"
 		(layer "F.Cu")
-		(at 91.44 95.25)
+		(at 91.44 96.52)
 		(descr "Mounting Hole 3.2mm, M3")
 		(tags "mounting hole 3.2mm m3")
@@
 	)
 	(gr_line
-		(start 87.63 107.95)
-		(end 87.63 115.57)
+		(start 87.63 109.22)
+		(end 87.63 116.84)
 		(stroke
 			(width 0.15)
@@
 	)
 	(gr_line
-		(start 87.63 57.15)
-		(end 88.265 57.15)
+		(start 87.63 58.42)
+		(end 88.265 58.42)
 		(stroke
 			(width 0.15)
@@
 	)
 	(gr_line
-		(start 87.757 125.73)
-		(end 88.392 125.73)
+		(start 87.757 127)
+		(end 88.392 127)
 		(stroke
 			(width 0.15)
@@
 	)
 	(gr_line
-		(start 87.63 59.69)
-		(end 87.63 67.31)
+		(start 87.63 60.96)
+		(end 87.63 68.58)
 		(stroke
 			(width 0.15)
@@
 	)
 	(gr_line
-		(start 87.63 49.53)
-		(end 87.63 57.15)
+		(start 87.63 50.8)
+		(end 87.63 58.42)
 		(stroke
 			(width 0.15)
@@
 	)
 	(gr_line
-		(start 87.63 115.57)
-		(end 88.265 115.57)
+		(start 87.63 116.84)
+		(end 88.265 116.84)
 		(stroke
 			(width 0.15)
@@
 	)
 	(gr_line
-		(start 88.265 59.69)
-		(end 87.63 59.69)
+		(start 88.265 60.96)
+		(end 87.63 60.96)
 		(stroke
 			(width 0.15)
@@
 	)
 	(gr_line
-		(start 88.392 118.11)
-		(end 87.757 118.11)
+		(start 88.392 119.38)
+		(end 87.757 119.38)
 		(stroke
 			(width 0.15)
@@
 	)
 	(gr_line
-		(start 88.265 107.95)
-		(end 87.63 107.95)
+		(start 88.265 109.22)
+		(end 87.63 109.22)
 		(stroke
 			(width 0.15)
@@
 	)
 	(gr_line
-		(start 88.265 49.53)
-		(end 87.63 49.53)
+		(start 88.265 50.8)
+		(end 87.63 50.8)
 		(stroke
 			(width 0.15)
@@
 	)
 	(gr_line
-		(start 87.757 118.11)
-		(end 87.757 125.73)
+		(start 87.757 119.38)
+		(end 87.757 127)
 		(stroke
 			(width 0.15)
@@
 	)
 	(gr_line
-		(start 87.63 67.31)
-		(end 88.265 67.31)
+		(start 87.63 68.58)
+		(end 88.265 68.58)
 		(stroke
 			(width 0.15)
@@
 	)
 	(gr_text "GND"
-		(at 84.074 112.014 0)
+		(at 84.074 113.284 0)
 		(layer "F.SilkS")
 		(effects
@@
 	)
 	(gr_text "\nInput"
-		(at 96.012 130.048 0)
+		(at 96.012 131.318 0)
 		(layer "F.SilkS")
 		(effects
@@
 	)
 	(gr_text "+5V"
-		(at 84.074 53.975 0)
+		(at 84.074 55.245 0)
 		(layer "F.SilkS")
 		(effects
@@
 	)
 	(gr_text "GND"
-		(at 84.074 64.1096 0)
+		(at 84.074 65.3796 0)
 		(layer "F.SilkS")
 		(effects
@@
 	)
 	(gr_text "+5V"
-		(at 84.074 122.428 0)
+		(at 84.074 123.698 0)
 		(layer "F.SilkS")
 		(effects
@@
 	)
 	(gr_text "\nOutput"
-		(at 95.25 46.228 0)
+		(at 95.25 47.498 0)
 		(layer "F.SilkS")
 		(effects
@@
 	)
 	(segment
-		(start 95.885 127.635)
-		(end 92.71 130.81)
+		(start 95.885 128.905)
+		(end 92.71 132.08)
 		(width 0.25)
 		(layer "F.Cu")
@@
 	)
 	(segment
-		(start 90.17 44.45)
-		(end 91.345 45.625)
+		(start 90.17 45.72)
+		(end 91.345 46.895)
 		(width 0.25)
 		(layer "F.Cu")
@@
 	)
 	(segment
-		(start 91.345 45.625)
-		(end 93.885 45.625)
+		(start 91.345 46.895)
+		(end 93.885 46.895)
 		(width 0.25)
 		(layer "F.Cu")
@@
 	)
 	(segment
-		(start 95.885 47.625)
-		(end 95.885 127.635)
+		(start 95.885 48.895)
+		(end 95.885 128.905)
 		(width 0.25)
 		(layer "F.Cu")
@@
 	)
 	(segment
-		(start 93.885 45.625)
-		(end 95.885 47.625)
+		(start 93.885 46.895)
+		(end 95.885 48.895)
 		(width 0.25)
 		(layer "F.Cu")
@@
 	)
 	(segment
-		(start 92.71 46.99)
-		(end 95.885 50.165)
+		(start 92.71 48.26)
+		(end 95.885 51.435)
 		(width 0.25)
 		(layer "B.Cu")
@@
 	)
 	(segment
-		(start 95.885 124.216701)
-		(end 93.101701 127)
+		(start 95.885 125.486701)
+		(end 93.101701 128.27)
 		(width 0.25)
 		(layer "B.Cu")
@@
 	)
 	(segment
-		(start 95.885 50.165)
-		(end 95.885 124.216701)
+		(start 95.885 51.435)
+		(end 95.885 125.486701)
 		(width 0.25)
 		(layer "B.Cu")
@@
 	)
 	(segment
-		(start 93.101701 127)
-		(end 91.44 127)
+		(start 93.101701 128.27)
+		(end 91.44 128.27)
 		(width 0.25)
 		(layer "B.Cu")
@@
 	)
 	(segment
-		(start 91.44 127)
-		(end 90.17 128.27)
+		(start 91.44 128.27)
+		(end 90.17 129.54)
 		(width 0.25)
 		(layer "B.Cu")
@@
 	)
 	(segment
-		(start 91.345 131.985)
-		(end 90.17 130.81)
+		(start 91.345 133.255)
+		(end 90.17 132.08)
 		(width 0.25)
 		(layer "F.Cu")
@@
 	)
 	(segment
-		(start 92.71 44.45)
-		(end 94.615 44.45)
+		(start 92.71 45.72)
+		(end 94.615 45.72)
 		(width 0.25)
 		(layer "F.Cu")
@@
 	)
 	(segment
-		(start 93.196701 131.985)
-		(end 91.345 131.985)
+		(start 93.196701 133.255)
+		(end 91.345 133.255)
 		(width 0.25)
 		(layer "F.Cu")
@@
 	)
 	(segment
-		(start 94.615 44.45)
-		(end 96.52 46.355)
+		(start 94.615 45.72)
+		(end 96.52 47.625)
 		(width 0.25)
 		(layer "F.Cu")
@@
 	)
 	(segment
-		(start 96.52 46.355)
-		(end 96.52 128.661701)
+		(start 96.52 47.625)
+		(end 96.52 129.931701)
 		(width 0.25)
 		(layer "F.Cu")
@@
 	)
 	(segment
-		(start 96.52 128.661701)
-		(end 93.196701 131.985)
+		(start 96.52 129.931701)
+		(end 93.196701 133.255)
 		(width 0.25)
 		(layer "F.Cu")
@@
 	)
 	(segment
-		(start 96.52 124.46)
-		(end 92.71 128.27)
+		(start 96.52 125.73)
+		(end 92.71 129.54)
 		(width 0.25)
 		(layer "B.Cu")
@@
 	)
 	(segment
-		(start 91.3638 45.7962)
-		(end 93.177901 45.7962)
+		(start 91.3638 47.0662)
+		(end 93.177901 47.0662)
 		(width 0.25)
 		(layer "B.Cu")
@@
 	)
 	(segment
-		(start 90.17 46.99)
-		(end 91.3638 45.7962)
+		(start 90.17 48.26)
+		(end 91.3638 47.0662)
 		(width 0.25)
 		(layer "B.Cu")
@@
 	)
 	(segment
-		(start 96.52 49.138299)
-		(end 96.52 124.46)
+		(start 96.52 50.408299)
+		(end 96.52 125.73)
 		(width 0.25)
 		(layer "B.Cu")
@@
 	)
 	(segment
-		(start 93.177901 45.7962)
-		(end 96.52 49.138299)
+		(start 93.177901 47.0662)
+		(end 96.52 50.408299)
 		(width 0.25)
 		(layer "B.Cu")

Commit message: ALSO ready to be sent
Parts:
- moved H2 1.27 mm to (91.4, 97.8)
- moved H3 1.27 mm to (91.4, 80.0)
Changed lines of the file:
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@@
 	(footprint "MountingHole:MountingHole_3.2mm_M3_Pad"
 		(layer "F.Cu")
-		(at 91.44 78.74)
+		(at 91.44 80.01)
 		(descr "Mounting Hole 3.2mm, M3")
 		(tags "mounting hole 3.2mm m3")
@@
 	(footprint "MountingHole:MountingHole_3.2mm_M3_Pad"
 		(layer "F.Cu")
-		(at 91.44 96.52)
+		(at 91.44 97.79)
 		(descr "Mounting Hole 3.2mm, M3")
 		(tags "mounting hole 3.2mm m3")
@@
 	)
 	(gr_text "EGS 1006 \nConnector"
-		(at 63.5 81.788 180)
+		(at 95.25 85.09 180)
 		(layer "F.SilkS")
 		(effects
@@
 	)
 	(gr_text "EGS 1006 \nConnector"
-		(at 55.88 88.9 0)
-		(layer "F.SilkS")
-		(effects
+		(at 87.63 92.202 0)
+		(layer "F.SilkS")
+		(effects

Commit message: check this
Parts:
- added J2: Conn_01x02_Pin, Connector_AMASS:AMASS_XT60PW-F_1x02_P7.20mm_Horizontal, F.Cu at (79.7, 123.6)
Other:
- board size 18 x 119.4 mm -> 30.7 x 119.4 mm

Commit message: jhkjlk
Parts:
- moved J2 68.6 mm to (79.7, 55.0)
Changed lines of the file:
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@@
 	(footprint "Connector_AMASS:AMASS_XT60PW-F_1x02_P7.20mm_Horizontal"
 		(layer "F.Cu")
-		(at 79.66 123.61 90)
+		(at 79.66 55.03 90)
 		(descr "Connector XT60 Horizontal PCB Female, https://www.tme.eu/en/Document/9b8d0c5eb7094295f3d3112c214d3ade/XT60PW%20SPEC.pdf")
 		(tags "RC Connector XT60")
