File: Wooden_Mirror.kicad_pcb (KiCad board)
At the start: 2 copper layers, 18 x 119.4 mm, 6 parts, among them J1 Conn_02x10_Odd_Even, J5 Conn_02x10_Odd_Even

Commit message: check connector
Parts:
- added J2: Conn_01x02_Pin, Connector_AMASS:AMASS_XT60PW-F_1x02_P7.20mm_Horizontal, F.Cu at (101.2, 80.4)
Routing:
- net GND: track 0.00 -> 31.9 mm
- net +5V: track 0.00 -> 19.4 mm
Other:
- board size 18 x 119.4 mm -> 31.8 x 119.4 mm

Commit message: update
Parts:
- moved J2 69.0 mm to (96.9, 149.2), turned to -90 degrees
Routing:
- net GND: track 31.9 -> 0.00 mm
- net +5V: track 19.4 -> 0.00 mm
Changed lines of the file:
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@@
 	(footprint "Connector_AMASS:AMASS_XT60PW-F_1x02_P7.20mm_Horizontal"
 		(layer "F.Cu")
-		(at 101.25 80.43 90)
+		(at 96.87 149.25 -90)
 		(descr "Connector XT60 Horizontal PCB Female, https://www.tme.eu/en/Document/9b8d0c5eb7094295f3d3112c214d3ade/XT60PW%20SPEC.pdf")
 		(tags "RC Connector XT60")
@@
 		)
 		(property "Footprint" "Connector_AMASS:AMASS_XT60PW-F_1x02_P7.20mm_Horizontal"
-			(at 0 0 90)
+			(at 0 0 -90)
 			(unlocked yes)
 			(layer "F.Fab")
@@
 		)
 		(property "Datasheet" ""
-			(at 0 0 90)
+			(at 0 0 -90)
 			(unlocked yes)
 			(layer "F.Fab")
@@
 		)
 		(property "Description" "Generic connector, single row, 01x02, script generated"
-			(at 0 0 90)
+			(at 0 0 -90)
 			(unlocked yes)
 			(layer "F.Fab")
@@
 		(attr through_hole)
 		(fp_line
+			(start -6.05 1.96)
+			(end -2.31 1.96)
+			(stroke
+				(width 0.12)
+				(type solid)
+			)
+			(layer "F.SilkS")
+		)
+		(fp_line
+			(start -11.46 -7.76)
+			(end -11.46 -2.15)
+			(stroke
+				(width 0.12)
+				(type solid)
+			)
+			(layer "F.SilkS")
+		)
+		(fp_line
+			(start -11.46 -7.76)
+			(end -10.61 -7.76)
+			(stroke
+				(width 0.12)
+				(type solid)
+			)
+			(layer "F.SilkS")
+		)
+		(fp_line
+			(start 3.41 -7.76)
+			(end 4.26 -7.76)
+			(stroke
+				(width 0.12)
+				(type solid)
+			)
+			(layer "F.SilkS")
+		)
+		(fp_line
+			(start 4.26 -7.76)
+			(end 4.26 -2.15)
+			(stroke
+				(width 0.12)
+				(type solid)
+			)
+			(layer "F.SilkS")
+		)
+		(fp_line
+			(start -10.61 -15.46)
+			(end -10.61 -7.76)
+			(stroke
+				(width 0.12)
+				(type solid)
+			)
+			(layer "F.SilkS")
+		)
+		(fp_line
+			(start -10.61 -15.46)
+			(end 3.41 -15.46)
+			(stroke
+				(width 0.12)
+				(type solid)
+			)
+			(layer "F.SilkS")
+		)
+		(fp_line
 			(start 3.41 -15.46)
 			(end 3.41 -7.76)
@@
 			(layer "F.SilkS")
 		)
-		(fp_line
-			(start -10.61 -15.46)
-			(end 3.41 -15.46)
-			(stroke
-				(width 0.12)
-				(type solid)
-			)
-			(layer "F.SilkS")
-		)
-		(fp_line
-			(start -10.61 -15.46)
-			(end -10.61 -7.76)
-			(stroke
-				(width 0.12)
-				(type solid)
-			)
-			(layer "F.SilkS")
-		)
-		(fp_line
-			(start 4.26 -7.76)
-			(end 4.26 -2.15)
-			(stroke
-				(width 0.12)
-				(type solid)
-			)
-			(layer "F.SilkS")
-		)
-		(fp_line
-			(start 3.41 -7.76)
-			(end 4.26 -7.76)
-			(stroke
-				(width 0.12)
-				(type solid)
-			)
-			(layer "F.SilkS")
-		)
-		(fp_line
-			(start -11.46 -7.76)
-			(end -10.61 -7.76)
-			(stroke
-				(width 0.12)
-				(type solid)
-			)
-			(layer "F.SilkS")
-		)
-		(fp_line
-			(start -11.46 -7.76)
+		(fp_arc
+			(start -8.5899 1.808718)
+			(mid -10.677645 0.302568)
 			(end -11.46 -2.15)
-			(stroke
-				(width 0.12)
-				(type solid)
-			)
-			(layer "F.SilkS")
-		)
-		(fp_line
-			(start -6.05 1.96)
-			(end -2.31 1.96)
 			(stroke
 				(width 0.12)
@@
 			(layer "F.SilkS")
 		)
-		(fp_arc
-			(start -8.5899 1.808718)
-			(mid -10.677645 0.302568)
-			(end -11.46 -2.15)
-			(stroke
-				(width 0.12)
-				(type solid)
-			)
-			(layer "F.SilkS")
+		(fp_line
+			(start 4.65 2.55)
+			(end -11.85 2.55)
+			(stroke
+				(width 0.05)
+				(type solid)
+			)
+			(layer "F.CrtYd")
+		)
+		(fp_line
+			(start 4.65 2.55)
+			(end 4.65 -15.85)
+			(stroke
+				(width 0.05)
+				(type solid)
+			)
+			(layer "F.CrtYd")
+		)
+		(fp_line
+			(start -11.85 -15.85)
+			(end -11.85 2.55)
+			(stroke
+				(width 0.05)
+				(type solid)
+			)
+			(layer "F.CrtYd")
 		)
 		(fp_line
@@
 		)
 		(fp_line
-			(start -11.85 -15.85)
-			(end -11.85 2.55)
-			(stroke
-				(width 0.05)
-				(type solid)
-			)
-			(layer "F.CrtYd")
-		)
-		(fp_line
-			(start 4.65 2.55)
-			(end 4.65 -15.85)
-			(stroke
-				(width 0.05)
-				(type solid)
-			)
-			(layer "F.CrtYd")
-		)
-		(fp_line
-			(start 4.65 2.55)
-			(end -11.85 2.55)
-			(stroke
-				(width 0.05)
-				(type solid)
-			)
-			(layer "F.CrtYd")
+			(start -7.35 1.85)
+			(end 0.15 1.85)
+			(stroke
+				(width 0.1)
+				(type solid)
+			)
+			(layer "F.Fab")
+		)
+		(fp_line
+			(start -11.35 -7.65)
+			(end -11.35 -2.15)
+			(stroke
+				(width 0.1)
+				(type solid)
+			)
+			(layer "F.Fab")
+		)
+		(fp_line
+			(start -11.35 -7.65)
+			(end 4.15 -7.65)
+			(stroke
+				(width 0.1)
+				(type solid)
+			)
+			(layer "F.Fab")
+		)
+		(fp_line
+			(start -10.5 -7.65)
+			(end -10.5 -15.35)
+			(stroke
+				(width 0.1)
+				(type solid)
+			)
+			(layer "F.Fab")
+		)
+		(fp_line
+			(start 3.3 -7.65)
+			(end 3.3 -15.35)
+			(stroke
+				(width 0.1)
+				(type solid)
+			)
+			(layer "F.Fab")
+		)
+		(fp_line
+			(start 4.15 -7.65)
+			(end 4.15 -2.15)
+			(stroke
+				(width 0.1)
+				(type solid)
+			)
+			(layer "F.Fab")
 		)
 		(fp_line
@@
 			(layer "F.Fab")
 		)
-		(fp_line
-			(start 4.15 -7.65)
-			(end 4.15 -2.15)
-			(stroke
-				(width 0.1)
-				(type solid)
-			)
-			(layer "F.Fab")
-		)
-		(fp_line
-			(start 3.3 -7.65)
-			(end 3.3 -15.35)
-			(stroke
-				(width 0.1)
-				(type solid)
-			)
-			(layer "F.Fab")
-		)
-		(fp_line
-			(start -10.5 -7.65)
-			(end -10.5 -15.35)
-			(stroke
-				(width 0.1)
-				(type solid)
-			)
-			(layer "F.Fab")
-		)
-		(fp_line
-			(start -11.35 -7.65)
-			(end 4.15 -7.65)
-			(stroke
-				(width 0.1)
-				(type solid)
-			)
-			(layer "F.Fab")
-		)
-		(fp_line
-			(start -11.35 -7.65)
+		(fp_arc
+			(start -7.385 1.885)
+			(mid -10.203176 0.688678)
 			(end -11.35 -2.15)
-			(stroke
-				(width 0.1)
-				(type solid)
-			)
-			(layer "F.Fab")
-		)
-		(fp_line
-			(start -7.35 1.85)
-			(end 0.15 1.85)
 			(stroke
 				(width 0.1)
@@
 			(layer "F.Fab")
 		)
-		(fp_arc
-			(start -7.385 1.885)
-			(mid -10.203176 0.688678)
-			(end -11.35 -2.15)
-			(stroke
-				(width 0.1)
-				(type solid)
-			)
-			(layer "F.Fab")
-		)
 		(fp_text user "-"
-			(at 2.8 2.5 90)
+			(at -10.82 2.5 90)
 			(layer "F.SilkS")
 			(effects
@@
 		)
 		(fp_text user "+"
-			(at -9.5 2.5 90)
+			(at 4.039 2.4836 90)
 			(layer "F.SilkS")
 			(effects
@@
 		)
 		(pad "" thru_hole rect
-			(at -10.35 -6 90)
+			(at -10.35 -6 270)
 			(size 0.9 2)
 			(drill oval 0.6 1.7)
@@
 		)
 		(pad "" thru_hole rect
-			(at 3.15 -6 90)
+			(at 3.15 -6 270)
 			(size 0.9 2)
 			(drill oval 0.6 1.7)
@@
 		)
 		(pad "1" thru_hole roundrect
-			(at 0 0 90)
+			(at 0 0 270)
 			(size 4.1 4.1)
 			(drill 2.7)
@@
 		)
 		(pad "2" thru_hole circle
-			(at -7.2 0 90)
+			(at -7.2 0 270)
 			(size 4.1 4.1)
 			(drill 2.7)
@@
 	)
 	(segment
-		(start 103.625 85.255)
-		(end 103.625 78.838796)
-		(width 0.25)
-		(layer "B.Cu")
-		(net 1)
-	)
-	(segment
-		(start 100.986204 76.2)
-		(end 82.55 76.2)
-		(width 0.25)
-		(layer "B.Cu")
-		(net 1)
-	)
-	(segment
-		(start 103.625 78.838796)
-		(end 100.986204 76.2)
-		(width 0.25)
-		(layer "B.Cu")
-		(net 1)
-	)
-	(segment
-		(start 101.25 87.63)
-		(end 103.625 85.255)
-		(width 0.25)
-		(layer "B.Cu")
-		(net 1)
-	)
-	(segment
 		(start 86.36 95.25)
 		(end 82.55 91.44)
@@
 		(layer "B.Cu")
 		(net 2)
-	)
-	(segment
-		(start 84.24 80.43)
-		(end 82.55 78.74)
-		(width 0.25)
-		(layer "B.Cu")
-		(net 3)
-	)
-	(segment
-		(start 101.25 80.43)
-		(end 84.24 80.43)
-		(width 0.25)
-		(layer "B.Cu")
-		(net 3)
 	)
 	(segment
@@
 		(polygon
 			(pts
-				(xy 73.914 52.578) (xy 74.041 171.195697) (xy 91.44 171.195697) (xy 91.44 52.578)
+				(xy 73.914 52.578) (xy 74.041 171.195697) (xy 104.14 171.195697) (xy 104.14 52.578)
 			)
 		)
@@
 		(polygon
 			(pts
-				(xy 73.914 52.578) (xy 74.041 171.195932) (xy 91.44 171.196) (xy 91.44 52.578)
-			)
-		)
+				(xy 73.914 52.578) (xy 74.041 171.195932) (xy 104.14 171.196) (xy 104.14 52.578)
+			)
+		)

Commit message: bfgdfs
Parts:
- moved J2 85.7 mm to (150.0, 81.9)
- moved H3 50.8 mm to (132.1, 55.9)
- moved H4 50.8 mm to (132.1, 101.6)
- moved H5 50.8 mm to (132.1, 119.4)
- moved H6 50.8 mm to (132.1, 165.1)
- moved J1 50.8 mm to (133.3, 153.7)
- moved J5 50.8 mm to (130.8, 67.3)
Other:
- board size 31.8 x 119.4 mm -> 92.7 x 120.6 mm
Changed lines of the file:
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@@
 	(footprint "MountingHole:MountingHole_3.2mm_M3_Pad"
 		(layer "F.Cu")
-		(at 81.28 120.65)
+		(at 132.08 119.38)
 		(descr "Mounting Hole 3.2mm, M3")
 		(tags "mounting hole 3.2mm m3")
@@
 	(footprint "Connector_PinHeader_2.54mm:PinHeader_2x10_P2.54mm_Vertical"
 		(layer "F.Cu")
-		(at 82.55 154.94 180)
+		(at 133.35 153.67 180)
 		(descr "Through hole straight pin header, 2x10, 2.54mm pitch, double rows")
 		(tags "Through hole pin header THT 2x10 2.54mm double row")
@@
 	(footprint "Connector_AMASS:AMASS_XT60PW-F_1x02_P7.20mm_Horizontal"
 		(layer "F.Cu")
-		(at 96.87 149.25 -90)
+		(at 149.956 81.94 -90)
 		(descr "Connector XT60 Horizontal PCB Female, https://www.tme.eu/en/Document/9b8d0c5eb7094295f3d3112c214d3ade/XT60PW%20SPEC.pdf")
 		(tags "RC Connector XT60")
@@
 	(footprint "MountingHole:MountingHole_3.2mm_M3_Pad"
 		(layer "F.Cu")
-		(at 81.28 166.37)
+		(at 132.08 165.1)
 		(descr "Mounting Hole 3.2mm, M3")
 		(tags "mounting hole 3.2mm m3")
@@
 	(footprint "Connector_PinHeader_2.54mm:PinHeader_2x10_P2.54mm_Vertical"
 		(layer "F.Cu")
-		(at 80.01 68.58)
+		(at 130.81 67.31)
 		(descr "Through hole straight pin header, 2x10, 2.54mm pitch, double rows")
 		(tags "Through hole pin header THT 2x10 2.54mm double row")
@@
 	(footprint "MountingHole:MountingHole_3.2mm_M3_Pad"
 		(layer "F.Cu")
-		(at 81.28 102.87)
+		(at 132.08 101.6)
 		(descr "Mounting Hole 3.2mm, M3")
 		(tags "mounting hole 3.2mm m3")
@@
 	(footprint "MountingHole:MountingHole_3.2mm_M3_Pad"
 		(layer "F.Cu")
-		(at 81.28 57.15)
+		(at 132.08 55.88)
 		(descr "Mounting Hole 3.2mm, M3")
 		(tags "mounting hole 3.2mm m3")
@@
 		(layer "F.SilkS")
 	)
+	(gr_line
+		(start 158.75 170.18)
+		(end 152.908 170.18)
+		(stroke
+			(width 0.1)
+			(type default)
+		)
+		(layer "Edge.Cuts")
+	)
 	(gr_rect
 		(start 73.66 52.07)
@@
 		)
 		(fill none)
+		(layer "Edge.Cuts")
+	)
+	(gr_line
+		(start 105.41 87.884)
+		(end 105.41 71.374)
+		(stroke
+			(width 0.1)
+			(type default)
+		)
+		(layer "Edge.Cuts")
+	)
+	(gr_line
+		(start 112.776 71.374)
+		(end 105.41 71.374)
+		(stroke
+			(width 0.1)
+			(type default)
+		)
+		(layer "Edge.Cuts")
+	)
+	(gr_line
+		(start 158.75 70.104)
+		(end 166.116 70.104)
+		(stroke
+			(width 0.1)
+			(type default)
+		)
+		(layer "Edge.Cuts")
+	)
+	(gr_line
+		(start 166.37 70.104)
+		(end 166.37 86.614)
+		(stroke
+			(width 0.1)
+			(type default)
+		)
+		(layer "Edge.Cuts")
+	)
+	(gr_line
+		(start 158.75 50.8)
+		(end 158.75 70.104)
+		(stroke
+			(width 0.1)
+			(type default)
+		)
+		(layer "Edge.Cuts")
+	)
+	(gr_line
+		(start 127 50.8)
+		(end 158.75 50.8)
+		(stroke
+			(width 0.1)
+			(type default)
+		)
+		(layer "Edge.Cuts")
+	)
+	(gr_line
+		(start 152.908 170.18)
+		(end 153.035 170.18)
+		(stroke
+			(width 0.1)
+			(type default)
+		)
+		(layer "Edge.Cuts")
+	)
+	(gr_line
+		(start 166.37 86.614)
+		(end 158.75 86.614)
+		(stroke
+			(width 0.1)
+			(type default)
+		)
+		(layer "Edge.Cuts")
+	)
+	(gr_line
+		(start 105.41 87.884)
+		(end 112.776 87.884)
+		(stroke
+			(width 0.1)
+			(type default)
+		)
+		(layer "Edge.Cuts")
+	)
+	(gr_line
+		(start 152.4 170.18)
+		(end 152.908 170.18)
+		(stroke
+			(width 0.1)
+			(type default)
+		)
+		(layer "Edge.Cuts")
+	)
+	(gr_line
+		(start 127 50.8)
+		(end 127 170.18)
+		(stroke
+			(width 0.1)
+			(type default)
+		)
+		(layer "Edge.Cuts")
+	)
+	(gr_line
+		(start 112.776 87.884)
+		(end 112.776 71.374)
+		(stroke
+			(width 0.1)
+			(type default)
+		)
+		(layer "Edge.Cuts")
+	)
+	(gr_line
+		(start 158.75 86.614)
+		(end 158.75 170.18)
+		(stroke
+			(width 0.1)
+			(type default)
+		)
+		(layer "Edge.Cuts")
+	)
+	(gr_line
+		(start 166.116 70.104)
+		(end 166.37 70.104)
+		(stroke
+			(width 0.1)
+			(type default)
+		)
+		(layer "Edge.Cuts")
+	)
+	(gr_line
+		(start 127 170.18)
+		(end 152.4 170.18)
+		(stroke
+			(width 0.1)
+			(type default)
+		)
 		(layer "Edge.Cuts")
 	)
@@
 			)
 		)
+	)
+	(zone
+		(net 3)
+		(net_name "+5V")
+		(layer "F.Cu")
+		(hatch edge 0.5)
+		(priority 2)
+		(connect_pads
+			(clearance 0.5)
+		)
+		(min_thickness 0.25)
+		(filled_areas_thickness no)
+		(fill
+			(thermal_gap 0.5)
+			(thermal_bridge_width 0.5)
+		)
+		(polygon
+			(pts
+				(xy 127.508 51.308) (xy 127.508 169.672) (xy 153.67 170.942) (xy 153.67 52.578)
+			)
+		)

Commit message: update
Parts:
- moved J2 0.29 mm to (150.0, 82.2)
Routing:
- net /Serial_IN: track 55.0 -> 51.4 mm
- net /LED_DIN: track 49.6 -> 46.6 mm
Other:
- board size 92.7 x 120.6 mm -> 39.4 x 119.4 mm
- board text removed: "EGS 1006 Connector"
- board text removed: "Input"
- board text removed: "Output"

Commit message: final
Other:
- board text added: "Input"
- board text added: "Output"
Changed lines of the file:
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@@
 		(layer "Edge.Cuts")
+	)
+	(gr_text "Output"
+		(at 137.668 89.408 0)
+		(layer "F.SilkS")
+		(effects
+			(font
+				(size 1 1)
+				(thickness 0.15)
+			)
+			(justify left bottom)
+		)
 	)
 	(gr_text "GND"
@@
 		(layer "F.SilkS")
 		(effects
+			(font
+				(size 1 1)
+				(thickness 0.15)
+			)
+			(justify left bottom)
+		)
+	)
+	(gr_text "Input"
+		(at 137.668 132.842 0)
+		(layer "F.SilkS")
+		(effects
