File: Wooden_Mirror.kicad_sch (KiCad schematic)
At the start: 2 parts, among them J1 Conn_02x10_Odd_Even, J5 Conn_02x10_Odd_Even

Commit message: nkmlkl
Parts:
- added H1, H2, H3, H4: MH, MountingHole:MountingHole_3.2mm_M3_Pad, symbol Mechanical:MountingHole_Pad
Connections:
- net GND: now also H1.1, H2.1, H3.1, H4.1

Commit message: check this
Parts:
- added J2: Conn_01x02_Pin, Connector_AMASS:AMASS_XT60PW-F_1x02_P7.20mm_Horizontal, symbol Connector:Conn_01x02_Pin
Connections:
- net +5V: now also J2.1 (Pin_1)
- net GND: now also J2.2 (Pin_2)
